File: kicad_files/athena.kicad_sch (KiCad schematic)
At the start: 557 parts, among them J1 TYPE-C-31-M-12, J2 A1001WR-S-04P, J3 SM04B-SRSS-TB(LF)(SN), Q1 2N7002, Q2 2N7002, Q3 AO3401A, Q4 2N7002, Q5 2N7002, SW1 K2-1187SQ-A4SW-06, SW10 MX Switch, SW100 MX Switch, SW101 MX Switch, SW102 MX Switch, SW103 MX Switch, SW104 MX Switch, SW105 MX Switch, SW106 MX Switch, SW107 MX Switch, SW108 MX Switch, SW109 MX Switch, SW11 MX Switch, SW110 MX Switch, SW111 MX Switch, SW112 MX Switch, SW113 MX Switch, SW12 MX Switch, SW13 MX Switch, SW14 MX Switch, SW15 MX Switch, SW16 MX Switch, SW17 MX Switch, SW18 MX Switch, SW19 MX Switch, SW2 MX Switch, SW20 MX Switch, SW21 MX Switch, SW22 MX Switch, SW23 MX Switch, SW24 MX Switch, SW25 MX Switch, SW26 MX Switch, SW27 MX Switch, SW28 MX Switch, SW29 MX Switch, SW3 MX Switch, SW30 MX Switch, SW31 MX Switch, SW32 MX Switch, SW33 MX Switch, SW34 MX Switch, SW35 MX Switch, SW36 MX Switch, SW37 MX Switch, SW38 MX Switch, SW39 MX Switch, SW4 MX Switch, SW40 MX Switch, SW41 MX Switch, SW42 MX Switch, SW43 MX Switch, SW44 MX Switch, SW45 MX Switch, SW46 MX Switch, SW47 MX Switch, SW48 MX Switch, SW49 MX Switch, SW5 MX Switch, SW50 MX Switch, SW51 MX Switch, SW52 MX Switch, SW53 MX Switch, SW54 MX Switch, SW55 MX Switch, SW56 MX Switch, SW57 MX Switch, SW58 MX Switch, SW59 MX Switch, SW6 MX Switch, SW60 MX Switch, SW61 MX Switch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

Commit message: First gamma version modifications
Parts:
- removed C20, C9: 1u, Capacitor_SMD:C_0805_2012Metric, symbol Device:C
- removed D3: SMF6.0A, acheron_Components:D_SOD-123, symbol Device:D_Schottky
- removed H1: DB_RGB_PASSTHROUGH_HOLE, athena_library:rgb_daughterboard_notch_plated_8x4mm, symbol Mechanical:MountingHole_Pad
- removed J3: SM04B-SRSS-TB(LF)(SN), acheron_Connectors:SM04B-SRSS-TB(LF)(SN)_mounting-reliefs, symbol Connector_Generic_MountingPin:Conn_01x04_MountingPin
- removed X7: RGB_PINS, acheron_Connectors:PinHeader_1x3_staggered_P2.54mm_Vertical, symbol Connector_Generic:Conn_01x03
- added D129, D130, D131, D132, D133: 1N4148W, acheron_Components:D_SOD-123, symbol Device:D
- added SW114, SW115, SW116, SW117, SW118: MX Switch, acheron_MX_SolderMask:MX100, symbol acheronSymbols:Mechanical_Switch
- SW60: Keycode END -> N2
- SW61: Keycode PGDN -> N3
- SW76: Keycode DEL -> N1
Connections:
- net C0: now also SW62.1, SW77.2; no longer SW62.2, SW77.1
- net C12: now also SW41.1
- net C14: now also SW114.2, SW118.2; no longer SW41.1
- net C15: now also SW115.1
- net C16: now also SW116.1, SW117.1
- net R1: now also D85.1 (K); no longer D68.1 (K)
- net R2: now also D102.1 (K); no longer D85.1 (K)
- net R3: now also D129.1 (K), D130.1 (K), D131.1 (K); no longer D102.1 (K)
- net R4: now also D132.1 (K), D133.1 (K)
- net R5: now also D68.1 (K)
- net RGB_5V_DB: no longer D36.1 (DOUT)
- net RGB_5V_MAIN: now also D21.3 (DIN); no longer D4.3 (DIN)
- net at D20.1 (DOUT): no longer D21.3 (DIN)
- new net: D133.2 (A), SW118.1
- new net: D131.2 (A), SW116.2
- new net: D88.2 (A), SW62.2, SW77.1
- new net: D132.2 (A), SW117.2
- new net: D129.2 (A), SW114.1
- new net: D130.2 (A), SW115.2
Other:
- moved on the sheet: C10, C11, C38, C39, C40, C41, C42, C43, C44, C45, C46, C47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

Commit message: Some routing
Parts:
- removed C52, C53: 100n, Capacitor_SMD:C_0805_2012Metric, symbol Device:C_Small
- added C20, C9: 100n, Capacitor_SMD:C_0402_1005Metric, symbol Device:C_Small
- added FB3: 4.7u, Inductor_SMD:L_1008_2520Metric, symbol Device:FerriteBead
- added GR10, GR11, GR12: Warning, acheron_Graphics:Warning_Sign_3.6x3.2mm, symbol Mechanical:MountingHole
- added LED113, LED114: LED, acheron_Components:LED_THT_2.54mm, symbol acheron_Symbols:LED
- added R118, R119, R120, R121, R122, R123, R124, R125, R126, R127, R128, R129, R130, R131, R132, R133: 5.1R, Resistor_SMD:R_0402_1005Metric, symbol Device:R_Small
- added R134, R135: 1k, Resistor_SMD:R_0805_2012Metric, symbol Device:R_Small
- added SW119, SW120: MX Switch, acheron_MX_SolderMask:MX200, symbol acheronSymbols:Mechanical_Switch
- C38, C39, C40, C41, C42, C43, C44, C45, C46, C47, C48, C49, C50, C51: footprint Capacitor_SMD:C_0805_2012Metric -> Capacitor_SMD:C_0402_1005Metric; Manufacturer Part Number CL21B104KCFNNNE -> CL05B104KB54PNC; Package C0805 -> C0402; Specification 100V 100nF X7R ±10% 0805 MLCC -> 50V 100nF X7R ±10% 0402 MLCC; Vendor Part Number LCSC C28233 -> LCSC C307331
Connections:
- net 5V: now also R118.2, R119.2, R120.2, R121.2, R122.2, R123.2, R124.2, R125.2, R126.2, R127.2, R128.2, R129.2, R130.2, R131.2, R132.2, R133.2; no longer C38.1, C39.1, C40.1, C41.1, C42.1, C43.1, C44.1, C45.1, C46.1, C47.1, C48.1, C49.1, C50.1, C51.1, D21.4 (VDD), D22.4 (VDD), D23.4 (VDD), D24.4 (VDD), D25.4 (VDD), D26.4 (VDD), D27.4 (VDD), D28.4 (VDD), D29.4 (VDD), D30.4 (VDD), D31.4 (VDD), D32.4 (VDD), D33.4 (VDD), D34.4 (VDD), D35.4 (VDD), D36.4 (VDD)
- net C14: now also SW119.1
- net C16: now also SW120.1
- net GND: now also LED63.K, LED64.K, LED65.K, LED66.K, R26.2, R45.2, R63.1, R79.2, R89.2, R90.2, C20.2, C9.2, LED113.K, LED114.K; no longer LED15.K, LED36.K, LED56.K, LED74.K, LED92.K, LED93.K, R83.2, R84.2, R85.2, R86.2
- net VBUS: now also FB3.1; no longer F1.2
- net at LED1.A, LED2.A, LED26.A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: now also LED15.A, LED36.A, LED56.A, LED74.A, LED92.A, LED93.A, R58.2, R59.2, R60.2, R61.2, R62.2, R64.2, R65.2, R66.2, R67.2, R83.1, R84.1, R85.1, R86.1, R134.1, R135.1; no longer LED63.A, LED64.A, LED65.A, LED66.A, R26.1, R45.1, R58.1, R59.1, R60.1, R61.1, R62.1, R63.1, R64.1, R65.1, R66.1, R67.1, R79.1, R89.1, R90.1
- net at LED55.A: now also R62.1; no longer R62.2
- net at LED52.A: now also R59.1; no longer R59.2
- net at R63.2: now also LED56.K; no longer LED56.A
- net at LED57.A: now also R64.1; no longer R64.2
- net at LED54.A: now also R61.1; no longer R61.2
- net at D128.2 (A), SW106.2: now also SW120.2
- net at LED58.A: now also R65.1; no longer R65.2
- net at LED59.A: now also R66.1; no longer R66.2
- net at D126.2 (A), SW104.1: now also SW119.2
- net at LED60.A: now also R67.1; no longer R67.2
- net at LED53.A: now also R60.1; no longer R60.2
- net at LED51.A: now also R58.1; no longer R58.2
- new net: C44.1, D29.4 (VDD), R126.1
- new net: C47.1, D32.4 (VDD), R129.1
- new net: F1.2, FB3.2
- new net: LED114.A, R135.2
- new net: C20.1, D21.4 (VDD), R118.1
- new net: C42.1, D27.4 (VDD), R124.1
- new net: C48.1, D33.4 (VDD), R130.1
- new net: C51.1, D36.4 (VDD), R133.1
- new net: LED113.A, R134.2
- new net: LED74.K, R79.1
- new net: LED93.K, R90.1
- new net: C39.1, D24.4 (VDD), R121.1
- new net: C50.1, D35.4 (VDD), R132.1
- new net: C40.1, D25.4 (VDD), R122.1
- new net: C45.1, D30.4 (VDD), R127.1
- new net: C38.1, D23.4 (VDD), R120.1
- new net: C43.1, D28.4 (VDD), R125.1
- new net: C41.1, D26.4 (VDD), R123.1
- new net: LED65.A, R85.2
- new net: C9.1, D22.4 (VDD), R119.1
- new net: C46.1, D31.4 (VDD), R128.1
- new net: LED66.A, R86.2
- new net: LED92.K, R89.1
- new net: LED15.K, R26.1
- new net: LED63.A, R83.2
- new net: LED64.A, R84.2
- new net: LED36.K, R45.1
- new net: C49.1, D34.4 (VDD), R131.1
Other:
- moved on the sheet: C12, C21, C22, C23, C24, C25, C26, C27, C28, C29, C30, C31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

Commit message: More routing
Parts:
- removed R134, R135: 1k, Resistor_SMD:R_0805_2012Metric, symbol Device:R_Small
- added LED115, LED116, LED117, LED118, LED119: LED, acheron_Components:LED_THT_2.54mm, symbol acheron_Symbols:LED
- added Q6, Q7, Q8: 2N7002, Package_TO_SOT_SMD:SOT-23, symbol Transistor_FET:2N7002
- added R136, R139, R142: 100R, Resistor_SMD:R_0805_2012Metric, symbol Device:R_Small
- added R137, R140, R143: 10k, Resistor_SMD:R_0805_2012Metric, symbol Device:R_Small
- added R138, R141, R144, R145, R146: 1k, Resistor_SMD:R_0805_2012Metric, symbol Device:R_Small
Connections:
- net C0: no longer U3.38 (USART6_RX/TIM3_CH2/PC7)
- net C1: now also SW63.2; no longer SW63.1, U3.37 (I2S2_MCK/TIM3_CH1/USART6_TX/PC6)
- net C10: no longer U3.20 (PA4/USART2_CK)
- net C11: no longer U3.17 (PA3/TIM2_CH4/USART2_RX)
- net C12: no longer U3.16 (PA2/TIM2_CH3/USART2_TX)
- net C13: no longer U3.25 (PC5)
- net C14: no longer U3.43 (USART1_RX/TIM1_CH3/PA10)
- net C15: no longer U3.41 (USART1_CK/TIM1_CH1/PA8)
- net C16: no longer U3.40 (TIM3_CH4/I2S_CKIN/PC9)
- net C2: no longer U3.35 (SPI2_MISO/PB14)
- net C3: no longer U3.33 (PB12)
- net C4: no longer U3.29 (PB10/TIM2_CH3/SPI2_SCK/I2C2_SCL/I2S2_CK)
- net C5: no longer U3.27 (PB1/TIM3_CH4)
- net C6: no longer U3.24 (PC4)
- net C7: no longer U3.23 (PA7/SPI1_MOSI/TIM3_CH2)
- net C8: no longer U3.22 (PA6/TIM3_CH1/SPI1_MISO)
- net C9: no longer U3.21 (PA5/TIM2_CH1/SPI1_SCK)
- net CAPS_INDICATOR: no longer U3.39 (USART6_CK/TIM3_CH3/PC8)
- net E-PA0: no longer U3.14 (PA0/TIM2_CH1/USART2_CTS)
- net E-PB3: no longer U3.55 (JTDO-SWO/SPI1_SCK/SPI3_SCK/I2C2_SDA/TIM2_CH2/PB3)
- net E-PB4: no longer U3.56 (NJTRST/SPI1_MISO/SPI3_MISO/I2C3_SDA/TIM3_CH1/PB4)
- net E-PB5: no longer U3.57 (SPI1_MOSI/SPI3_MOSI/TIM3_CH2/PB5)
- net E-PB8: no longer U3.61 (I2C1_SCL/TIM4_CH3/TIM10_CH1/PB8)
- net E-PB9: no longer U3.62 (I2C1_SDA/TIM4_CH4/TIM11_CH1/PB9)
- net E-PC1: no longer U3.9 (PC1)
- net E-PC2: no longer U3.10 (PC2/SPI2_MISO)
- net E-PC3: no longer U3.11 (PC3/SPI2_MOSI)
- net E-PD2: no longer U3.54 (PD2)
- net GND: now also LED118.K, LED119.K, Q6.2 (S), Q7.2 (S), Q8.2 (S), R137.1, R138.2, R140.1, R141.2, R143.1, R144.2; no longer R37.2, R53.2, R55.2
- net LED_PWM: now also U3.40 (TIM3_CH4/I2S_CKIN/PC9); no longer U3.26 (PB0/TIM3_CH3)
- net R0: no longer U3.52 (SPI3_MISO/PC11)
- net R1: no longer U3.53 (SPI3_MOSI/PC12)
- net R2: no longer U3.51 (SPI3_SCK/I2S3_CK/PC10)
- net R3: no longer U3.50 (JTDI/TIM2_CH1/PA14)
- net R4: no longer U3.8 (PC0)
- net R5: no longer U3.15 (PA1/TIM2_CH2/USART2_RTS)
- net LED_PWM_OUT: now reaches LED1.A, LED15.A, LED2.A, LED27.A, LED28.A, LED36.A, LED4.A, LED45.A, LED46.A, LED47.A, LED48.A, LED56.A, LED67.A, LED74.A, LED78.A, LED79.A, LED80.A, LED81.A, LED82.A, LED83.A, LED84.A, LED85.A, LED86.A, LED87.A, LED88.A, LED89.A, LED90.A, LED91.A, LED92.A, LED93.A, LED95.A, Q3.3 (D), R107.1, R108.1, R109.1, R110.1, R111.1, R112.1, R113.1, R114.1, R116.1, R20.1, R21.1, R22.1, R23.2, R24.2, R25.1, R27.1, R28.1, R29.1, R30.1, R31.1, R32.1, R38.1, R39.1, R40.1, R41.1, R42.1, R43.1, R44.1, R46.1, R47.1, R48.1, R49.1, R50.1, R51.1, R52.1, R56.1, R57.1, R58.2, R59.2, R60.2, R61.2, R62.2, R64.2, R65.2, R66.2, R67.2, R68.1, R69.1, R74.1, R75.1, R76.1, R77.1, R78.1, R80.1, R81.1, R82.1, R83.1, R84.1, R85.1, R86.1, R91.1
- net LED_PWM_OUT: now also R115.2, R37.1, R53.2, LED115.A, LED116.A, LED117.A, R145.1, R146.1; no longer LED26.A, LED3.A, R115.1
- net at LED114.A: now also LED111.A, R115.1
- net at LED28.K: now also R55.2; no longer R55.1
- net at LED113.A: now also LED112.A, R116.2
- net at D89.2 (A): now also SW63.1; no longer SW63.2
- net at LED3.K: now also Q8.3 (D); no longer R37.1
- net at R53.1: now also LED26.A; no longer LED26.K
- new net: LED118.A, R145.2
- new net: LED116.K, R141.1
- new net: Q7.1 (G), R139.2, R140.2
- new net: Q7.3 (D), R55.1
- new net: Q6.1 (G), R136.2, R137.2
- new net: Q8.1 (G), R142.2, R143.2
- new net: LED3.A, R37.2
- new net: LED115.K, R138.1
- new net: LED26.K, Q6.3 (D)
- new net: LED119.A, R146.2
- new net: LED117.K, R144.1
- new net NUM_INDICATOR_1: R136.1
- new net NUM_INDICATOR_2: R139.1
- new net SCROLL_INDICATOR: R142.1
Other:
- moved on the sheet: LED112, LED113, LED114, LED26, LED28, LED3, LED68, LED69, Q5, R116, R37, R53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

Commit message: More routing
Connections:
- net C1: now also U3.16 (PA2/TIM2_CH3/USART2_TX); no longer SW108.1, SW80.1, SW97.1
- net C10: now also U3.23 (PA7/SPI1_MOSI/TIM3_CH2)
- net C11: now also U3.22 (PA6/TIM3_CH1/SPI1_MISO)
- net C12: now also U3.21 (PA5/TIM2_CH1/SPI1_SCK)
- net C13: now also U3.20 (PA4/USART2_CK)
- net C14: now also U3.38 (USART6_RX/TIM3_CH2/PC7)
- net C15: now also U3.37 (I2S2_MCK/TIM3_CH1/USART6_TX/PC6)
- net C16: now also U3.35 (SPI2_MISO/PB14)
- net C4: now also U3.15 (PA1/TIM2_CH2/USART2_RTS)
- net C5: now also U3.29 (PB10/TIM2_CH3/SPI2_SCK/I2C2_SCL/I2S2_CK)
- net C6: now also U3.27 (PB1/TIM3_CH4)
- net C7: now also U3.26 (PB0/TIM3_CH3)
- net C8: now also U3.25 (PC5)
- net C9: now also U3.24 (PC4)
- net LED_PWM: now also U3.39 (USART6_CK/TIM3_CH3/PC8); no longer U3.40 (TIM3_CH4/I2S_CKIN/PC9)
- net R5: no longer D119.1 (K)
- new net C17: SW108.1, SW80.1, SW97.1, U3.40 (TIM3_CH4/I2S_CKIN/PC9)
Other:
- moved on the sheet: D104, D119, SW108, SW80, SW97

Commit message: More routing
Parts:
- removed X3: Conn_01x02, acheron_Connectors:PinHeader_1x3_staggered_P2.54mm_Vertical, symbol Connector_Generic:Conn_01x03
- removed X4: EXTRA_PINS, acheron_Connectors:PinHeader_2x3_P2.54mm_Vertical, symbol Connector_Generic:Conn_02x03_Odd_Even
- removed X5: EXTRA_PINS, acheron_Connectors:PinHeader_2x6_P2.54mm_Vertical, symbol Connector_Generic:Conn_02x06_Odd_Even
Connections:
- net C0: now also U3.50 (JTDI/TIM2_CH1/PA14)
- net C11: now also SW106.1, SW116.1, SW117.1, SW120.1, SW18.1, SW43.1, SW61.1
- net C12: now also SW105.1, SW115.1, SW17.1, SW42.1, SW60.1, SW93.1
- net C13: now also SW104.2, SW114.2, SW118.2, SW119.1, SW16.2, SW59.2, SW76.2
- net C14: now also SW108.1, SW80.1, SW97.1; no longer SW104.2, SW114.2, SW118.2, SW119.1, SW16.2, SW59.2, SW76.2, U3.38 (USART6_RX/TIM3_CH2/PC7)
- net C2: now also U3.11 (PC3/SPI2_MOSI)
- net C3: now also U3.14 (PA0/TIM2_CH1/USART2_CTS)
- net CAPS_INDICATOR: now also U3.43 (USART1_RX/TIM1_CH3/PA10)
- net LED_PWM: now also U3.38 (USART6_RX/TIM3_CH2/PC7); no longer U3.39 (USART6_CK/TIM3_CH3/PC8)
- net NUM_INDICATOR_1: now also U3.61 (I2C1_SCL/TIM4_CH3/TIM10_CH1/PB8)
- net NUM_INDICATOR_2: now also U3.8 (PC0)
- net R0: no longer D51.1 (K), D52.1 (K), D53.1 (K)
- net R1: no longer D69.1 (K), D70.1 (K), D85.1 (K)
- net R2: now also U3.17 (PA3/TIM2_CH4/USART2_RX); no longer D102.1 (K), D86.1 (K), D87.1 (K)
- net R3: no longer D129.1 (K), D130.1 (K), D131.1 (K)
- net R4: now also U3.41 (USART1_CK/TIM1_CH1/PA8); no longer D117.1 (K), D132.1 (K), D133.1 (K)
- net R5: now also D119.1 (K), U3.51 (SPI3_SCK/I2S3_CK/PC10); no longer D126.1 (K), D127.1 (K), D128.1 (K)
- net R9: now reaches U3.10 (PC2/SPI2_MISO)
- net R9: now also D69.1 (K), D70.1 (K), D85.1 (K)
- net R10: now reaches U3.9 (PC1)
- net R10: now also D102.1 (K), D86.1 (K), D87.1 (K)
- removed net C15: SW105.1, SW115.1, SW17.1, SW42.1, SW60.1, SW93.1, U3.37 (I2S2_MCK/TIM3_CH1/USART6_TX/PC6)
- removed net C16: SW106.1, SW116.1, SW117.1, SW120.1, SW18.1, SW43.1, SW61.1, U3.35 (SPI2_MISO/PB14)
- removed net C17: SW108.1, SW80.1, SW97.1, U3.40 (TIM3_CH4/I2S_CKIN/PC9)
- new net R11: D129.1 (K), D130.1 (K), D131.1 (K), U3.39 (USART6_CK/TIM3_CH3/PC8)
- new net R6: D117.1 (K), D132.1 (K), D133.1 (K), U3.37 (I2S2_MCK/TIM3_CH1/USART6_TX/PC6)
- new net R7: D126.1 (K), D127.1 (K), D128.1 (K), U3.40 (TIM3_CH4/I2S_CKIN/PC9)
- new net R8: D51.1 (K), D52.1 (K), D53.1 (K), U3.35 (SPI2_MISO/PB14)
Other:
- moved on the sheet: D102, D103, D104, D105, D106, D107, D108, D109, D110, D111, D112, D113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

Commit message: More routing
Connections:
- net R2: no longer D71.1 (K)
- net R12: now reaches U3.62 (I2C1_SDA/TIM4_CH4/TIM11_CH1/PB9)
- net R12: now also D71.1 (K)
Other:
- moved on the sheet: D71, SW45
Changed lines of the file:
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@@
   (junction (at 327.66 717.55) (diameter 0.9144) (color 0 0 0 0)
   )
-  (junction (at 69.85 603.25) (diameter 1.016) (color 0 0 0 0)
-  )
   (junction (at 920.75 635) (diameter 0) (color 0 0 0 0)
   )
@@
   (junction (at 222.25 565.15) (diameter 1.016) (color 0 0 0 0)
   )
+  (junction (at 69.85 717.55) (diameter 0) (color 0 0 0 0)
+  )
   (junction (at 749.3 603.25) (diameter 0.9144) (color 0 0 0 0)
   )
@@
   (junction (at 336.55 615.95) (diameter 1.016) (color 0 0 0 0)
   )
-  (junction (at 82.55 577.85) (diameter 1.016) (color 0 0 0 0)
-  )
   (junction (at 311.15 365.125) (diameter 0.9144) (color 0 0 0 0)
   )
@@
     (stroke (width 0) (type solid))
   )
-  (wire (pts (xy 82.55 590.55) (xy 82.55 594.36))
+  (wire (pts (xy 82.55 971.55) (xy 82.55 975.36))
     (stroke (width 0) (type solid))
   )
@@
     (stroke (width 0) (type solid))
   )
+  (wire (pts (xy 57.15 958.85) (xy 82.55 958.85))
+    (stroke (width 0) (type solid))
+  )
   (wire (pts (xy 996.95 603.25) (xy 1016 603.25))
     (stroke (width 0) (type solid))
@@
     (stroke (width 0) (type solid))
   )
-  (wire (pts (xy 107.95 577.85) (xy 82.55 577.85))
+  (wire (pts (xy 57.15 577.85) (xy 107.95 577.85))
     (stroke (width 0) (type solid))
   )
@@
     (stroke (width 0) (type solid))
   )
+  (wire (pts (xy 69.85 717.55) (xy 69.85 984.25))
+    (stroke (width 0) (type default))
+  )
   (wire (pts (xy 844.55 676.91) (xy 844.55 678.18))
     (stroke (width 0) (type solid))
@@
     (stroke (width 0) (type solid))
   )
-  (wire (pts (xy 69.85 603.25) (xy 73.66 603.25))
+  (wire (pts (xy 69.85 984.25) (xy 73.66 984.25))
     (stroke (width 0) (type solid))
   )
@@
     (stroke (width 0) (type solid))
   )
-  (wire (pts (xy 57.15 577.85) (xy 82.55 577.85))
-    (stroke (width 0) (type solid))
-  )
   (wire (pts (xy 1028.7 716.915) (xy 1041.4 716.915))
     (stroke (width 0) (type default))
@@
     (stroke (width 0) (type solid))
   )
-  (wire (pts (xy 69.85 641.35) (xy 69.85 603.25))
+  (wire (pts (xy 69.85 565.15) (xy 69.85 641.35))
     (stroke (width 0) (type solid))
   )
@@
     (stroke (width 0) (type default))
   )
-  (wire (pts (xy 82.55 577.85) (xy 82.55 582.93))
+  (wire (pts (xy 82.55 958.85) (xy 82.55 963.93))
     (stroke (width 0) (type solid))
   )
@@
     (stroke (width 0) (type solid))
   )
-  (wire (pts (xy 69.85 603.25) (xy 69.85 565.15))
-    (stroke (width 0) (type solid))
-  )
   (wire (pts (xy 387.35 552.45) (xy 387.35 556.26))
     (stroke (width 0) (type solid))
@@
     )
   )
+  (global_label "R12" (shape input) (at 57.15 958.85 180)
+    (effects (font (size 1.27 1.27)) (justify right))
+    (property "Intersheetrefs" "${INTERSHEET_REFS}" (at 31.75 722.63 0)
+      (effects (font (size 1.27 1.27)) hide)
+    )
+  )
   (global_label "BOOT0" (shape input) (at 236.855 43.815 90)
     (effects (font (size 1.27 1.27)) (justify left))
@@
     )
   )
+  (global_label "R12" (shape input) (at 224.155 43.815 90)
+    (effects (font (size 1.27 1.27)) (justify left))
+    (property "Intersheetrefs" "${INTERSHEET_REFS}" (at 460.375 18.415 0)
+      (effects (font (size 1.27 1.27)) hide)
+    )
+  )
   (global_label "DBUS-" (shape bidirectional) (at 820.42 46.99 0)
     (effects (font (size 1.27 1.27)) (justify left))
@@
     )
   )
-  (symbol (lib_id "Device:D") (at 82.55 586.74 270) (unit 1)
+  (symbol (lib_id "Device:D") (at 82.55 967.74 270) (unit 1)
     (in_bom yes) (on_board yes) (dnp no)
-    (property "Reference" "D71" (at 88.0302 586.74 0)
+    (property "Reference" "D71" (at 88.0302 967.74 0)
       (effects (font (size 1.27 1.27)))
     )
-    (property "Value" "1N4148W" (at 85.7315 586.74 0)
+    (property "Value" "1N4148W" (at 85.7315 967.74 0)
       (effects (font (size 1.27 1.27)))
     )
-    (property "Footprint" "acheron_Components:D_SOD-123" (at 82.55 586.74 0)
+    (property "Footprint" "acheron_Components:D_SOD-123" (at 82.55 967.74 0)
       (effects (font (size 1.27 1.27)) hide)
     )
-    (property "Datasheet" "~" (at 82.55 586.74 0)
+    (property "Datasheet" "~" (at 82.55 967.74 0)
       (effects (font (size 1.27 1.27)) hide)
     )
-    (property "Package" "SOD-123" (at 82.55 586.74 0)
+    (property "Package" "SOD-123" (at 82.55 967.74 0)
       (effects (font (size 1.27 1.27)) hide)
     )
-    (property "Specification" "Small-signal switching diodes" (at 82.55 586.74 0)
+    (property "Specification" "Small-signal switching diodes" (at 82.55 967.74 0)
       (effects (font (size 1.27 1.27)) hide)
     )
-    (property "Description" "" (at 82.55 586.74 0)
+    (property "Description" "" (at 82.55 967.74 0)
       (effects (font (size 1.27 1.27)) hide)
     )
-    (property "Manufacturer" "Semtech" (at 82.55 586.74 0)
+    (property "Manufacturer" "Semtech" (at 82.55 967.74 0)
       (effects (font (size 1.27 1.27)) hide)
     )
-    (property "Manufacturer Part Number" "1N4148W" (at 82.55 586.74 0)
+    (property "Manufacturer Part Number" "1N4148W" (at 82.55 967.74 0)
       (effects (font (size 1.27 1.27)) hide)
     )
-    (property "Vendor Part Number" "LCSC C81598" (at 82.55 586.74 0)
+    (property "Vendor Part Number" "LCSC C81598" (at 82.55 967.74 0)
       (effects (font (size 1.27 1.27)) hide)
     )
@@
     )
   )
-  (symbol (lib_id "acheronSymbols:Mechanical_Switch") (at 82.55 603.25 90) (mirror x) (unit 1)
+  (symbol (lib_id "acheronSymbols:Mechanical_Switch") (at 82.55 984.25 90) (mirror x) (unit 1)
     (in_bom yes) (on_board yes) (dnp no)
-    (property "Reference" "SW45" (at 82.55 602.615 90)
+    (property "Reference" "SW45" (at 82.55 983.615 90)
       (effects (font (size 1.27 1.27)))
     )
-    (property "Value" "MX Switch" (at 86.36 603.25 0)
+    (property "Value" "MX Switch" (at 86.36 984.25 0)
       (effects (font (size 0.762 0.762)) hide)
     )
-    (property "Footprint" "acheron_MX_SolderMask:MX150" (at 82.55 603.25 0)
+    (property "Footprint" "acheron_MX_SolderMask:MX150" (at 82.55 984.25 0)
       (effects (font (size 1.27 1.27)) hide)
     )
-    (property "Datasheet" "" (at 82.55 603.25 0)
+    (property "Datasheet" "" (at 82.55 984.25 0)
       (effects (font (size 1.27 1.27)) hide)
     )
-    (property "Keycode" "TAB" (at 82.55 604.52 90)
+    (property "Keycode" "TAB" (at 82.55 985.52 90)
       (effects (font (size 0.762 0.762)))
     )
-    (property "Manufacturer" "" (at 82.55 603.25 0)
+    (property "Manufacturer" "" (at 82.55 984.25 0)
       (effects (font (size 1.27 1.27)) hide)
     )
-    (property "Specification" "MX-style mechanical keyboard switch" (at 82.55 603.25 0)
+    (property "Specification" "MX-style mechanical keyboard switch" (at 82.55 984.25 0)
       (effects (font (size 1.27 1.27)) hide)
     )
-    (property "Description" "" (at 82.55 603.25 0)
+    (property "Description" "" (at 82.55 984.25 0)
       (effects (font (size 1.27 1.27)) hide)
     )

Commit message: Finished routing, DRC pending
Parts:
- added R134, R135, R147, R148, R149, R150, R151, R152, R153, R154, R155, R156, R157, R158, R159, R160, R161: 5.1R, Resistor_SMD:R_0402_1005Metric, symbol Device:R_Small
- C21, C22, C23, C24, C25, C26, C27, C28, C29, C30, C31, C32, C33, C34, C35, C36, C37: footprint Capacitor_SMD:C_0805_2012Metric -> Capacitor_SMD:C_0402_1005Metric; Manufacturer Part Number CL21B104KCFNNNE -> CL05B104KB54PNC; Package C0805 -> C0402; Specification 100V 100nF X7R ±10% 0805 MLCC -> 50V 100nF X7R ±10% 0402 MLCC; Vendor Part Number LCSC C28233 -> LCSC C307331
Connections:
- net E-PC14 is gone; now on net R0: U3.3 (PC14/OSC32_IN)
- net E-PC15 is gone; now on net R1: U3.4 (PC15/OSC32_OUT)
- net 5V: now also F1.2, R134.2, R135.2, R147.2, R148.2, R149.2, R150.2, R151.2, R152.2, R153.2, R154.2, R155.2, R156.2, R157.2, R158.2, R159.2, R160.2, R161.2; no longer C21.1, C22.1, C23.1, C24.1, C25.1, C26.1, C27.1, C28.1, C29.1, C30.1, C31.1, C32.1, C33.1, C34.1, C35.1, C36.1, C37.1, D10.4 (VDD), D11.4 (VDD), D12.4 (VDD), D13.4 (VDD), D14.4 (VDD), D15.4 (VDD), D16.4 (VDD), D17.4 (VDD), D18.4 (VDD), D19.4 (VDD), D20.4 (VDD), D4.4 (VDD), D5.4 (VDD), D6.4 (VDD), D7.4 (VDD), D8.4 (VDD), D9.4 (VDD), F1.1
- net SCROLL_INDICATOR: now also U3.33 (PB12)
- net at FB3.2: now also F1.1; no longer F1.2
- net at D36.1 (DOUT): now also D4.3 (DIN)
- new net: C25.1, D8.4 (VDD), R149.1
- new net: C31.1, D14.4 (VDD), R155.1
- new net: C30.1, D13.4 (VDD), R154.1
- new net: C23.1, D6.4 (VDD), R147.1
- new net: C35.1, D18.4 (VDD), R159.1
- new net: C32.1, D15.4 (VDD), R156.1
- new net: C34.1, D17.4 (VDD), R158.1
- new net: C36.1, D19.4 (VDD), R160.1
- new net: C21.1, D4.4 (VDD), R134.1
- new net: C22.1, D5.4 (VDD), R135.1
- new net: C37.1, D20.4 (VDD), R161.1
- new net: C24.1, D7.4 (VDD), R148.1
- new net: C27.1, D10.4 (VDD), R151.1
- new net: C33.1, D16.4 (VDD), R157.1
- new net: C29.1, D12.4 (VDD), R153.1
- new net: C26.1, D9.4 (VDD), R150.1
- new net: C28.1, D11.4 (VDD), R152.1
Other:
- moved on the sheet: F1
