File: kicad_files/athena.kicad_sch (KiCad schematic)
At the start: 620 parts, among them J1 TYPE-C-31-M-12, J2 A1001WR-S-04P, Q1 2N7002, Q2 2N7002, Q3 AO3401A, Q4 2N7002, Q5 2N7002, Q6 2N7002, Q7 2N7002, Q8 2N7002, SW1 K2-1187SQ-A4SW-06, SW10 MX Switch, SW100 MX Switch, SW101 MX Switch, SW102 MX Switch, SW103 MX Switch, SW104 MX Switch, SW105 MX Switch, SW106 MX Switch, SW107 MX Switch, SW108 MX Switch, SW109 MX Switch, SW11 MX Switch, SW110 MX Switch, SW111 MX Switch, SW112 MX Switch, SW113 MX Switch, SW114 MX Switch, SW115 MX Switch, SW116 MX Switch, SW117 MX Switch, SW118 MX Switch, SW119 MX Switch, SW12 MX Switch, SW120 MX Switch, SW13 MX Switch, SW14 MX Switch, SW15 MX Switch, SW16 MX Switch, SW17 MX Switch, SW18 MX Switch, SW19 MX Switch, SW2 MX Switch, SW20 MX Switch, SW21 MX Switch, SW22 MX Switch, SW23 MX Switch, SW24 MX Switch, SW25 MX Switch, SW26 MX Switch, SW27 MX Switch, SW28 MX Switch, SW29 MX Switch, SW3 MX Switch, SW30 MX Switch, SW31 MX Switch, SW32 MX Switch, SW33 MX Switch, SW34 MX Switch, SW35 MX Switch, SW36 MX Switch, SW37 MX Switch, SW38 MX Switch, SW39 MX Switch, SW4 MX Switch, SW40 MX Switch, SW41 MX Switch, SW42 MX Switch, SW43 MX Switch, SW44 MX Switch, SW45 MX Switch, SW46 MX Switch, SW47 MX Switch, SW48 MX Switch, SW49 MX Switch, SW5 MX Switch, SW50 MX Switch, SW51 MX Switch, SW52 MX Switch, SW53 MX Switch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

Commit message: ESD improvement, tracing and labels
Parts:
- removed FB2: GZ2012D601TF, Inductor_SMD:L_0805_2012Metric, symbol Device:Ferrite_Bead_Small
Connections:
- net GND: no longer U1.2 (GND)
- net GNDPWR: now also U1.2 (GND), X6.1
Other:
- moved on the sheet: X6
Changed lines of the file:
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@@
     (stroke (width 0) (type solid))
   )
-  (wire (pts (xy 52.705 181.61) (xy 52.705 180.34))
+  (wire (pts (xy 50.8 181.61) (xy 50.8 184.15))
     (stroke (width 0) (type solid))
   )
@@
     (stroke (width 0) (type solid))
   )
-  (wire (pts (xy 1127.76 372.745) (xy 1111.25 372.745))
-    (stroke (width 0) (type solid))
-  )
   (wire (pts (xy 430.53 368.3) (xy 414.02 368.3))
     (stroke (width 0) (type solid))
@@
     (stroke (width 0) (type solid))
   )
-  (wire (pts (xy 52.705 187.96) (xy 52.705 186.69))
-    (stroke (width 0) (type solid))
-  )
   (wire (pts (xy 302.26 528.32) (xy 302.26 527.05))
     (stroke (width 0) (type solid))
@@
     )
   )
-  (global_label "RGB_5V_DB" (shape output) (at 1127.76 372.745 0)
-    (effects (font (size 2.54 2.54)) (justify left))
-    (property "Intersheetrefs" "${INTERSHEET_REFS}" (at 1133.4533 372.6974 0)
-      (effects (font (size 2.54 2.54)) (justify left) hide)
-    )
-  )
   (global_label "3V3" (shape input) (at 599.44 249.555 90)
     (effects (font (size 1.27 1.27)) (justify left))
@@
     )
   )
-  (symbol (lib_id "power:GND") (at 810.26 59.69 0) (unit 1)
-    (in_bom yes) (on_board yes) (dnp no)
-    (property "Reference" "#PWR012" (at 810.26 66.04 0)
-      (effects (font (size 1.27 1.27)) hide)
-    )
-    (property "Value" "GND" (at 810.26 63.5 0)
-      (effects (font (size 0.7874 0.7874)))
-    )
-    (property "Footprint" "" (at 810.26 59.69 0)
-      (effects (font (size 1.27 1.27)) hide)
-    )
-    (property "Datasheet" "" (at 810.26 59.69 0)
-      (effects (font (size 1.27 1.27)) hide)
-    )
-    (pin "1")
-    (instances
-      (project "athena"
-        (path "/9ce6b20d-0a6c-402a-b232-5eafd6242eb3"
-          (reference "#PWR012") (unit 1)
-        )
-      )
-    )
-  )
   (symbol (lib_id "power:GND") (at 844.55 685.8 0) (unit 1)
     (in_bom yes) (on_board yes) (dnp no)
@@
     )
   )
-  (symbol (lib_id "Device:Ferrite_Bead_Small") (at 52.705 184.15 0) (unit 1)
-    (in_bom yes) (on_board yes) (dnp no)
-    (property "Reference" "FB2" (at 56.1086 183.007 0)
-      (effects (font (size 1.27 1.27)) (justify left))
-    )
-    (property "Value" "GZ2012D601TF" (at 56.1086 185.293 0)
-      (effects (font (size 1.27 1.27)) (justify left))
-    )
-    (property "Footprint" "Inductor_SMD:L_0805_2012Metric" (at 50.927 184.15 90)
-      (effects (font (size 1.27 1.27)) hide)
-    )
-    (property "Datasheet" "~" (at 52.705 184.15 0)
-      (effects (font (size 1.27 1.27)) hide)
-    )
-    (property "Manufacturer" "Sunlord" (at 52.705 184.15 0)
-      (effects (font (size 1.27 1.27)) hide)
-    )
-    (property "Manufacturer Part Number" "GZ2012D601TF" (at 52.705 184.15 0)
-      (effects (font (size 1.27 1.27)) hide)
-    )
-    (property "LCSC Part Number" "" (at 52.705 184.15 0)
-      (effects (font (size 1.27 1.27)) hide)
-    )
-    (property "Package" "L0805" (at 52.705 184.15 0)
-      (effects (font (size 1.27 1.27)) hide)
-    )
-    (property "Specification" "600R @ 100MHz ferrite bead" (at 52.705 184.15 0)
-      (effects (font (size 1.27 1.27)) hide)
-    )
-    (property "Vendor Part Number" "LCSC C1017" (at 52.705 184.15 0)
-      (effects (font (size 1.27 1.27)) hide)
-    )
-    (pin "1")
-    (pin "2")
-    (instances
-      (project "athena"
-        (path "/9ce6b20d-0a6c-402a-b232-5eafd6242eb3"
-          (reference "FB2") (unit 1)
-        )
-      )
-    )
-  )
   (symbol (lib_id "acheronSymbols:Mechanical_Switch") (at 209.55 527.05 0) (unit 1)
     (in_bom yes) (on_board yes) (dnp no)
@@
     )
   )
+  (symbol (lib_id "power:GNDPWR") (at 810.26 59.69 0) (unit 1)
+    (in_bom yes) (on_board yes) (dnp no)
+    (property "Reference" "#PWR012" (at 810.26 64.77 0)
+      (effects (font (size 1.27 1.27)) hide)
+    )
+    (property "Value" "GNDPWR" (at 809.625 62.23 0)
+      (effects (font (size 0.508 0.508)))
+    )
+    (property "Footprint" "" (at 810.26 60.96 0)
+      (effects (font (size 1.27 1.27)) hide)
+    )
+    (property "Datasheet" "" (at 810.26 60.96 0)
+      (effects (font (size 1.27 1.27)) hide)
+    )
+    (pin "1")
+    (instances
+      (project "athena"
+        (path "/9ce6b20d-0a6c-402a-b232-5eafd6242eb3"
+          (reference "#PWR012") (unit 1)
+        )
+      )
+    )
+  )
   (symbol (lib_id "Device:D") (at 158.75 510.54 270) (unit 1)
     (in_bom yes) (on_board yes) (dnp no)
@@
     )
   )
+  (symbol (lib_id "power:GNDPWR") (at 50.8 184.15 0) (unit 1)
+    (in_bom yes) (on_board yes) (dnp no)
+    (property "Reference" "#PWR048" (at 50.8 189.23 0)
+      (effects (font (size 1.27 1.27)) hide)
+    )
+    (property "Value" "GNDPWR" (at 50.165 186.69 0)
+      (effects (font (size 0.508 0.508)))
+    )
+    (property "Footprint" "" (at 50.8 185.42 0)
+      (effects (font (size 1.27 1.27)) hide)
+    )
+    (property "Datasheet" "" (at 50.8 185.42 0)
+      (effects (font (size 1.27 1.27)) hide)
+    )
+    (pin "1")
+    (instances
+      (project "athena"
+        (path "/9ce6b20d-0a6c-402a-b232-5eafd6242eb3"
+          (reference "#PWR048") (unit 1)
+        )
+      )
+    )
+  )
   (symbol (lib_id "acheronSymbols:Mechanical_Switch") (at 412.75 679.45 90) (mirror x) (unit 1)
     (in_bom yes) (on_board yes) (dnp no)
@@
     )
   )
-  (symbol (lib_id "power:GND") (at 52.705 187.96 0) (unit 1)
-    (in_bom yes) (on_board yes) (dnp no)
-    (property "Reference" "#PWR048" (at 52.705 194.31 0)
-      (effects (font (size 1.27 1.27)) hide)
-    )
-    (property "Value" "GND" (at 52.705 191.77 0)
-      (effects (font (size 0.7874 0.7874)))
-    )
-    (property "Footprint" "" (at 52.705 187.96 0)
-      (effects (font (size 1.27 1.27)) hide)
-    )
-    (property "Datasheet" "" (at 52.705 187.96 0)
-      (effects (font (size 1.27 1.27)) hide)
-    )
-    (pin "1")
-    (instances
-      (project "athena"
-        (path "/9ce6b20d-0a6c-402a-b232-5eafd6242eb3"
-          (reference "#PWR048") (unit 1)
-        )
-      )
-    )
-  )
   (symbol (lib_id "acheron_Symbols:LED") (at 958.85 712.47 270) (unit 1)
     (in_bom no) (on_board yes) (dnp no) (fields_autoplaced)
@@
     )
   )
-  (symbol (lib_name "Mechanical:MountingHole_1") (lib_id "Mechanical:MountingHole_Pad") (at 52.705 177.8 0) (unit 1)
+  (symbol (lib_name "Mechanical:MountingHole_1") (lib_id "Mechanical:MountingHole_Pad") (at 50.8 179.07 0) (unit 1)
     (in_bom no) (on_board yes) (dnp no)
-    (property "Reference" "X6" (at 56.515 176.53 0)
+    (property "Reference" "X6" (at 54.61 177.8 0)
       (effects (font (size 1.27 1.27)) (justify left))
     )
-    (property "Value" "MountingHole" (at 56.515 179.07 0)
+    (property "Value" "MountingHole" (at 54.61 180.34 0)
       (effects (font (size 1.27 1.27)) (justify left))
     )
-    (property "Footprint" "MountingHole:MountingHole_2.5mm_Pad" (at 52.705 177.8 0)
+    (property "Footprint" "MountingHole:MountingHole_2.5mm_Pad" (at 50.8 179.07 0)
       (effects (font (size 1.27 1.27)) hide)
     )
-    (property "Datasheet" "~" (at 52.705 177.8 0)
+    (property "Datasheet" "~" (at 50.8 179.07 0)
       (effects (font (size 1.27 1.27)) hide)
     )
